Commit message: commit

File: src/description/gbot_description.urdf (robot description, URDF)
Before this commit: robot wam-v, 4 links, 3 joints
Links:
- added link camera_link
- link base_link: mass 180.0 -> None; geometry visual mesh filename=package://gbot_nav/models/GBOT-Base/mesh/gbot.dae
Joints:
- added joint camera_joint: type fixed, parent base_link, child camera_link, origin xyz=0.383 0 0.334 rpy=0 0 0
- joint imu_joint: origin xyz=0 0.0 0.944 rpy=0 0 0 -> xyz=0.3 0.191 0.272 rpy=0 0 0
- joint lidar_joint: origin xyz=0.701 0 1.031 rpy=0 0 0 -> xyz=0 0 0.363 rpy=0 0 0
